Commit message: fix gripper urdf

File: urdf/fr07_g101gm.xacro (robot description, xacro)
@@ -26,5 +26,5 @@
             <origin xyz="0 0 0" rpy="0 0 0" />
             <geometry>
-                <mesh filename="file://$(find fr07_g101gm)/meshes/gripper_main_link.stl" scale="0.001 0.001 0.001"/>
+                <mesh filename="file://$(find open_manipulator_pro_description)/meshes/gripper_main_link.stl" scale="0.001 0.001 0.001"/>
             </geometry>
             </collision>
@@ -32,5 +32,5 @@
             <origin xyz="0 0 0" rpy="0 0 0" />
             <geometry>
-                <mesh filename="file://$(find fr07_g101gm)/meshes/gripper_main_link.stl" scale="0.001 0.001 0.001"/>
+                <mesh filename="file://$(find open_manipulator_pro_description)/meshes/gripper_main_link.stl" scale="0.001 0.001 0.001"/>
             </geometry>
             <material name="grey"/>
@@ -59,5 +59,5 @@
             <origin xyz="0 0 0" rpy="0 0 0" />
             <geometry>
-                <mesh filename="file://$(find fr07_g101gm)/meshes/gripper_link.stl" scale="0.001 0.001 0.001"/>
+                <mesh filename="file://$(find open_manipulator_pro_description)/meshes/gripper_link.stl" scale="0.001 0.001 0.001"/>
             </geometry>
             <material name="grey"/>
@@ -66,5 +66,5 @@
             <origin xyz="0 0 0" rpy="0 0 0" />
             <geometry>
-                <mesh filename="file://$(find fr07_g101gm)/meshes/gripper_link.stl" scale="0.001 0.001 0.001"/>
+                <mesh filename="file://$(find open_manipulator_pro_description)/meshes/gripper_link.stl" scale="0.001 0.001 0.001"/>
             </geometry>
             <material name="grey"/>
@@ -93,5 +93,5 @@
             <origin xyz="0 0 0" rpy="0 0 0" />
             <geometry>
-                <mesh filename="file://$(find fr07_g101gm)/meshes/gripper_sub_link.stl" scale="0.001 0.001 0.001"/>
+                <mesh filename="file://$(find open_manipulator_pro_description)/meshes/gripper_sub_link.stl" scale="0.001 0.001 0.001"/>
             </geometry>
             <material name="grey"/>
@@ -100,5 +100,5 @@
             <origin xyz="0 0 0" rpy="0 0 0" />
             <geometry>
-                <mesh filename="file://$(find fr07_g101gm)/meshes/gripper_sub_link.stl" scale="0.001 0.001 0.001"/>
+                <mesh filename="file://$(find open_manipulator_pro_description)/meshes/gripper_sub_link.stl" scale="0.001 0.001 0.001"/>
             </geometry>
             <material name="grey"/>
